Commit message: Updating xacro script to ROS Kinetic

File: urdf/prsg2_description.xacro (robot description, xacro)
@@ -1,5 +1,5 @@
 <?xml version="1.0" encoding="UTF-8" ?>
 <robot name="prsg2_robot" xmlns:xacro="http://www.ros.org/wiki/xacro">
-  <xacro:property name="pi" value="3.14159" />
+  <!-- <xacro:property name="pi" value="3.14159" /> -->
   <xacro:property name="degree" value="${pi / 180}" />
   <xacro:property name="inch" value="0.0254" />
